File: schematic_pcb/electronic_design_kicad/memotype.pretty/electronic_design_kicad.kicad_pcb (KiCad board)
At the start: 2 copper layers, 34.3 x 18.2 mm, 20 parts, among them IC1 ATTINY85-S, P1 USB_A, P2 CONN_6

Commit message: first steps to memtype revision 2 pcb
Parts:
- moved R4 1.20 mm to (156.5, 177.7), turned to 180 degrees
- moved D1 0.85 mm to (150.0, 186.6)
- moved C1 0.20 mm to (161.5, 177.7), turned to 180 degrees
- moved R3 0.20 mm to (150.0, 182.9)
Routing:
- net /LEFT: track 0.00 -> 20.0 mm, vias 0 -> 1
- net +5V: track 32.7 -> 16.7 mm
- net DGND: track 40.9 -> 56.6 mm
- net D-: track 13.4 -> 8.61 mm
- net D+: track 8.25 -> 6.25 mm
Other:
- board size 34.3 x 18.2 mm -> 34.3 x 13.6 mm
