File: schematic_pcb/electronic_design_kicad/electronic_design_kicad.sch (KiCad schematic (older format))
At the start: 19 parts, among them IC1 ATTINY85-S, P1 USB_A, P2 CONN_6

Commit message: added 3d design files and finished schematic and PCB
Parts:
- C2: mouser C0805C104K5RACTU -> C0805C472K5RACTU
- D2: mouser (none) -> L29K-F2J1-24-Z
- D3: mouser (none) -> Q976-NR-1
- P1: mouser (none) -> 534-932
- P2: mouser (none) -> SKRHAAE010
- R10, R11: value 68R -> 220R; mouser ERJ-6GEYJ680V -> ERJ-6GEYJ221V
- R9: value 1M -> 560k
Other:
- note added: "Reset pin has a pull-up resistor.\nNo external one needed."
Changed lines of the file:
@@
 P 6250 1550
 F 0 "R9" V 6250 1650 40  0000 C CNN
-F 1 "1M" V 6250 1500 40  0000 C CNN
+F 1 "560k" V 6250 1500 40  0000 C CNN
 F 2 "projectLib:SMD-0805" V 6180 1550 30  0001 C CNN
-F 3 "~" H 6250 1550 30  0000 C CNN
+F 3 "" H 6250 1550 30  0000 C CNN
 F 4 "1/4W" V 6250 1550 40  0001 C CNN "Power"
 F 5 "ERJ-6GEYJ564V" V 6250 1550 60  0001 C CNN "mouser"
@@
 F 2 "projectLib:SMD-0805" H 6488 1400 30  0001 C CNN
 F 3 "~" H 6450 1550 60  0000 C CNN
-F 4 "C0805C104K5RACTU" H 6450 1550 60  0001 C CNN "mouser"
+F 4 "C0805C472K5RACTU" H 6450 1550 60  0001 C CNN "mouser"
 	1    6450 1550
 	1    0    0    -1
@@
 F 1 "CONN_6" V 7500 1700 50  0000 C CNN
 F 2 "projectLib:SKRHAAE010" H 7450 1750 60  0001 C CNN
-F 3 "" H 7450 1750 60  0000 C CNN
+F 3 "http://www.alps.com/products/WebObjects/catalog.woa/E/HTML/MultiControl/Switch/SKRH/SKRHAAE010.html" H 7450 1750 60  0001 C CNN
+F 4 "SKRHAAE010" V 7450 1750 60  0001 C CNN "mouser"
 	1    7450 1750
 	-1   0    0    1
@@
 F 1 "USB_A" H 5850 1600 50  0000 C CNN
 F 2 "projectLib:USB_A_MALE" H 5850 1300 60  0001 C CNN
-F 3 "" V 5850 1300 60  0000 C CNN
+F 3 "http://www.mouser.com/ds/2/215/32-744715.pdf" H 5850 1300 60  0001 C CNN
+F 4 "534-932" H 5900 1400 60  0001 C CNN "mouser"
 	1    5900 1400
 	1    0    0    -1
@@
 F 1 "LED GREEN" H 2650 3250 50  0000 C CNN
 F 2 "LEDs:LED_0603" H 2650 3350 60  0001 C CNN
-F 3 "" H 2650 3350 60  0000 C CNN
+F 3 "" H 2650 3350 60  0001 C CNN
+F 4 "L29K-F2J1-24-Z" H 2650 3350 60  0001 C CNN "mouser"
 	1    2650 3350
 	0    1    -1   0
@@
 F 1 "LED RED" H 2950 3250 50  0000 C CNN
 F 2 "LEDs:LED_0603" H 2950 3350 60  0001 C CNN
-F 3 "" H 2950 3350 60  0000 C CNN
+F 3 "" H 2950 3350 60  0001 C CNN
+F 4 "Q976-NR-1" H 2950 3350 60  0001 C CNN "mouser"
 	1    2950 3350
 	0    1    -1   0
@@
 P 2950 2850
 F 0 "R11" V 2950 2950 40  0000 C CNN
-F 1 "68R" V 2950 2800 40  0000 C CNN
+F 1 "220R" V 2950 2800 40  0000 C CNN
 F 2 "projectLib:SMD-0805" V 2880 2850 30  0001 C CNN
 F 3 "~" H 2950 2850 30  0000 C CNN
 F 4 "1/8W" V 2950 2850 40  0001 C CNN "Power"
-F 5 "ERJ-6GEYJ680V" V 2950 2850 60  0001 C CNN "mouser"
+F 5 "ERJ-6GEYJ221V" V 2950 2850 60  0001 C CNN "mouser"
 	1    2950 2850
 	1    0    0    -1
@@
 P 2650 2850
 F 0 "R10" V 2650 2950 40  0000 C CNN
-F 1 "68R" V 2650 2800 40  0000 C CNN
+F 1 "220R" V 2650 2800 40  0000 C CNN
 F 2 "projectLib:SMD-0805" V 2580 2850 30  0001 C CNN
 F 3 "~" H 2650 2850 30  0000 C CNN
 F 4 "1/8W" V 2650 2850 40  0001 C CNN "Power"
-F 5 "ERJ-6GEYJ680V" V 2650 2850 60  0001 C CNN "mouser"
+F 5 "ERJ-6GEYJ221V" V 2650 2850 60  0001 C CNN "mouser"
 	1    2650 2850
 	1    0    0    -1
@@
 Wire Wire Line
 	5100 1800 5100 1650
+Text Notes 1550 2600 0    60   ~ 0
+Reset pin has a pull-up resistor.\nNo external one needed.
 $EndSCHEMATC
