File: schematic_pcb/electronic_design_kicad/electronic_design_kicad.sch (KiCad schematic (older format))
At the start: 19 parts, among them IC1 ATTINY85-S, P1 USB_A, P2 CONN_6

Commit message: update joystick direction in schematic and code
Connections:
- net RIGHT is gone; now on net LEFT: P2.6, R7.2, R8.1
- net LEFT: no longer P2.3, R4.2, R6.1
- new net UP: P2.3, R4.2, R6.1
Changed lines of the file:
@@
 	8300 2850 8300 1450
 Text Label 7850 1950 0    60   ~ 0
+RIGHT
+Text Label 7850 1750 0    60   ~ 0
 UP
-Text Label 7850 1750 0    60   ~ 0
-LEFT
 Text Label 7850 1650 0    60   ~ 0
 DOWN
 Text Label 7850 1450 0    60   ~ 0
-RIGHT
+LEFT
 $Comp
 L R R9

Commit message: hardware revision 3.0
Parts:
- removed D2: LED GREEN, projectLib:LED_0603_PIPE, symbol LED
- removed R10: 220R, projectLib:SMD-0805, symbol R
- added R12: 1k, projectLib:SMD-0805, symbol R
Connections:
- net DGND: now also R12.2; no longer R8.2
- net CENTER: now reaches P2.2
- net CENTER: now also R8.2, R12.1
- net G: no longer names the net of IC1.5 (PB0(MOSI/DI/SDA/AIN0/OC0A/OC1A/AREF/PCINT0))
Other:
- note added: "Reset pin has internal pull-up resistor.\nNo external one needed."
- note removed: "Reset pin has a pull-up resistor.\nNo external one needed."
- moved on the sheet: D3, R11
Changed lines of the file:
@@
 Sheet 1 1
 Title "MemType PCB schematic"
-Date "2016-01-06"
-Rev "2"
+Date "2016-06-08"
+Rev "3"
 Comp "website: www.area0x33.com"
 Comment1 ""
@@
 $EndComp
 $Comp
-L DGND #PWR01
+L DGND #PWR5
 U 1 1 5432C0B8
 P 5100 2450
-F 0 "#PWR01" H 5100 2450 40  0001 C CNN
+F 0 "#PWR5" H 5100 2450 40  0001 C CNN
 F 1 "DGND" H 5100 2380 40  0000 C CNN
 F 2 "" H 5100 2450 60  0000 C CNN
@@
 $EndComp
 $Comp
-L +5V #PWR02
+L +5V #PWR4
 U 1 1 5432D97B
 P 5100 1650
-F 0 "#PWR02" H 5100 1740 20  0001 C CNN
+F 0 "#PWR4" H 5100 1740 20  0001 C CNN
 F 1 "+5V" H 5100 1740 30  0000 C CNN
 F 2 "" H 5100 1650 60  0000 C CNN
@@
 $EndComp
 $Comp
-L +5V #PWR03
+L +5V #PWR1
 U 1 1 5432D981
 P 1050 1350
-F 0 "#PWR03" H 1050 1440 20  0001 C CNN
+F 0 "#PWR1" H 1050 1440 20  0001 C CNN
 F 1 "+5V" H 1050 1440 30  0000 C CNN
 F 2 "" H 1050 1350 60  0000 C CNN
@@
 Connection ~ 1250 2100
 $Comp
-L DGND #PWR04
+L DGND #PWR2
 U 1 1 5432DBE1
 P 1150 2900
-F 0 "#PWR04" H 1150 2900 40  0001 C CNN
+F 0 "#PWR2" H 1150 2900 40  0001 C CNN
 F 1 "DGND" H 1150 2830 40  0000 C CNN
 F 2 "" H 1150 2900 60  0000 C CNN
@@
 	5800 1750 5800 1700
 $Comp
-L DGND #PWR05
+L DGND #PWR7
 U 1 1 5432DF65
 P 6000 1750
-F 0 "#PWR05" H 6000 1750 40  0001 C CNN
+F 0 "#PWR7" H 6000 1750 40  0001 C CNN
 F 1 "DGND" H 6000 1680 40  0000 C CNN
 F 2 "" H 6000 1750 60  0000 C CNN
@@
 $EndComp
 $Comp
-L +5V #PWR06
+L +5V #PWR6
 U 1 1 5432DF84
 P 5600 1750
-F 0 "#PWR06" H 5600 1840 20  0001 C CNN
+F 0 "#PWR6" H 5600 1840 20  0001 C CNN
 F 1 "+5V" H 5600 1840 30  0000 C CNN
 F 2 "" H 5600 1750 60  0000 C CNN
@@
 	8850 1250 8850 1200
 $Comp
-L +5V #PWR07
+L +5V #PWR10
 U 1 1 543DE636
 P 8850 1200
-F 0 "#PWR07" H 8850 1290 20  0001 C CNN
+F 0 "#PWR10" H 8850 1290 20  0001 C CNN
 F 1 "+5V" H 8850 1290 30  0000 C CNN
 F 2 "" H 8850 1200 60  0000 C CNN
@@
 	1    0    0    -1
 $EndComp
-Wire Wire Line
-	8850 3400 8850 3450
 Wire Wire Line
 	8850 2300 8650 2300
@@
 Microcontroller circuit and peripherals
 Wire Notes Line
-	6750 3700 9150 3700
-Wire Notes Line
-	6750 1050 6750 3700
-Wire Notes Line
-	9200 3700 9200 1050
+	6750 1050 6750 4100
+Wire Notes Line
+	9200 1050 9200 4100
 $Comp
 L ZENER_DUAL D1
@@
 	1050 2200 1050 2350
 $Comp
-L DGND #PWR08
+L DGND #PWR9
 U 1 1 546258D9
 P 8100 2600
-F 0 "#PWR08" H 8100 2600 40  0001 C CNN
+F 0 "#PWR9" H 8100 2600 40  0001 C CNN
 F 1 "DGND" H 8100 2530 40  0000 C CNN
 F 2 "" H 8100 2600 60  0000 C CNN
@@
 $EndComp
 $Comp
-L DGND #PWR09
+L DGND #PWR11
 U 1 1 5462598D
-P 8850 3450
-F 0 "#PWR09" H 8850 3450 40  0001 C CNN
-F 1 "DGND" H 8850 3380 40  0000 C CNN
-F 2 "" H 8850 3450 60  0000 C CNN
-F 3 "" H 8850 3450 60  0000 C CNN
-	1    8850 3450
+P 8850 3900
+F 0 "#PWR11" H 8850 3900 40  0001 C CNN
+F 1 "DGND" H 8850 3830 40  0000 C CNN
+F 2 "" H 8850 3900 60  0000 C CNN
+F 3 "" H 8850 3900 60  0000 C CNN
+	1    8850 3900
 	1    0    0    -1
 $EndComp
@@
 	6450 2000 6250 2000
 $Comp
-L DGND #PWR010
+L DGND #PWR8
 U 1 1 568C63F8
 P 6250 2100
-F 0 "#PWR010" H 6250 2100 40  0001 C CNN
+F 0 "#PWR8" H 6250 2100 40  0001 C CNN
 F 1 "DGND" H 6250 2030 40  0000 C CNN
 F 2 "" H 6250 2100 60  0000 C CNN
@@
 Wire Wire Line
 	8400 1950 7850 1950
-NoConn ~ 7850 1850
 $Comp
 L USB_A P1
@@
 $EndComp
 $Comp
-L LED D2
-U 1 1 56901E90
-P 3850 3350
-F 0 "D2" H 3850 3450 50  0000 C CNN
-F 1 "LED GREEN" H 3850 3250 50  0000 C CNN
-F 2 "projectLib:LED_0603_PIPE" H 3850 3350 60  0001 C CNN
-F 3 "" H 3850 3350 60  0001 C CNN
-F 4 "L29K-F2J1-24-Z" H 3850 3350 60  0001 C CNN "mouser"
-	1    3850 3350
-	0    1    -1   0
-$EndComp
-$Comp
-L DGND #PWR011
+L DGND #PWR3
 U 1 1 5690231F
-P 3850 3700
-F 0 "#PWR011" H 3850 3700 40  0001 C CNN
-F 1 "DGND" H 3850 3630 40  0000 C CNN
-F 2 "" H 3850 3700 60  0000 C CNN
-F 3 "" H 3850 3700 60  0000 C CNN
-	1    3850 3700
+P 3750 3600
+F 0 "#PWR3" H 3750 3600 40  0001 C CNN
+F 1 "DGND" H 3750 3530 40  0000 C CNN
+F 2 "" H 3750 3600 60  0000 C CNN
+F 3 "" H 3750 3600 60  0000 C CNN
+	1    3750 3600
 	1    0    0    -1
 $EndComp
@@
 L LED D3
 U 1 1 569024A8
-P 4150 3350
-F 0 "D3" H 4150 3450 50  0000 C CNN
-F 1 "LED RED" H 4150 3250 50  0000 C CNN
-F 2 "projectLib:LED_0603_PIPE" H 4150 3350 60  0001 C CNN
-F 3 "" H 4150 3350 60  0001 C CNN
-F 4 "Q976-NR-1" H 4150 3350 60  0001 C CNN "mouser"
-	1    4150 3350
+P 3750 3350
+F 0 "D3" H 3750 3450 50  0000 C CNN
+F 1 "LED RED" H 3750 3250 50  0000 C CNN
+F 2 "projectLib:LED_0603_PIPE" H 3750 3350 60  0001 C CNN
+F 3 "" H 3750 3350 60  0001 C CNN
+F 4 "Q976-NR-1" H 3750 3350 60  0001 C CNN "mouser"
+	1    3750 3350
 	0    1    -1   0
 $EndComp
 Wire Wire Line
-	2300 1900 2050 1900
-Wire Wire Line
-	2300 1800 2050 1800
-Wire Wire Line
-	3850 3550 3850 3700
-Wire Wire Line
-	3850 3600 4150 3600
-Wire Wire Line
-	4150 3600 4150 3550
-Connection ~ 3850 3600
+	3750 3600 3750 3550
 $Comp
 L R R11
 U 1 1 569034B6
-P 4150 2850
-F 0 "R11" V 4150 2950 40  0000 C CNN
-F 1 "220R" V 4150 2800 40  0000 C CNN
-F 2 "projectLib:SMD-0805" V 4080 2850 30  0001 C CNN
-F 3 "~" H 4150 2850 30  0000 C CNN
-F 4 "1/8W" V 4150 2850 40  0001 C CNN "Power"
-F 5 "ERJ-6GEYJ221V" V 4150 2850 60  0001 C CNN "mouser"
-	1    4150 2850
-	1    0    0    -1
-$EndComp
-$Comp
-L R R10
-U 1 1 5690360A
-P 3850 2850
-F 0 "R10" V 3850 2950 40  0000 C CNN
-F 1 "220R" V 3850 2800 40  0000 C CNN
-F 2 "projectLib:SMD-0805" V 3780 2850 30  0001 C CNN
-F 3 "~" H 3850 2850 30  0000 C CNN
-F 4 "1/8W" V 3850 2850 40  0001 C CNN "Power"
-F 5 "ERJ-6GEYJ221V" V 3850 2850 60  0001 C CNN "mouser"
-	1    3850 2850
-	1    0    0    -1
-$EndComp
-Wire Wire Line
-	4150 3100 4150 3150
-Wire Wire Line
-	3850 3100 3850 3150
-Text Label 4150 2600 0    60   ~ 0
+P 3750 2850
+F 0 "R11" V 3750 2950 40  0000 C CNN
+F 1 "220R" V 3750 2800 40  0000 C CNN
+F 2 "projectLib:SMD-0805" V 3680 2850 30  0001 C CNN
+F 3 "~" H 3750 2850 30  0000 C CNN
+F 4 "1/8W" V 3750 2850 40  0001 C CNN "Power"
+F 5 "ERJ-6GEYJ221V" V 3750 2850 60  0001 C CNN "mouser"
+	1    3750 2850
+	1    0    0    -1
+$EndComp
+Wire Wire Line
+	3750 3100 3750 3150
+Text Label 3750 2600 0    60   ~ 0
 R
-Text Label 3850 2600 0    60   ~ 0
-G
-Text Label 2050 1800 0    60   ~ 0
-G
+Wire Wire Line
+	5100 1800 5100 1650
+Text Notes 1800 2650 0    60   ~ 0
+Reset pin has internal pull-up resistor.\nNo external one needed.
+$Comp
+L R R12
+U 1 1 575737C3
+P 8850 3650
+F 0 "R12" V 8850 3750 40  0000 C CNN
+F 1 "1k" V 8850 3600 40  0000 C CNN
+F 2 "projectLib:SMD-0805" V 8780 3650 30  0001 C CNN
+F 3 "~" H 8850 3650 30  0000 C CNN
+F 4 "1/4W" V 8850 3650 40  0001 C CNN "Power"
+F 5 "ERJ-6GEYJ102V" V 8850 3650 60  0001 C CNN "mouser"
+	1    8850 3650
+	1    0    0    -1
+$EndComp
+Wire Notes Line
+	9200 4100 6750 4100
+Wire Wire Line
+	8850 3400 8500 3400
+Wire Wire Line
+	8500 3400 8500 1850
+Wire Wire Line
+	8500 1850 7850 1850
+Text Label 7850 1850 0    60   ~ 0
+CENTER
 Text Label 2050 1900 0    60   ~ 0
 R
 Wire Wire Line
-	5100 1800 5100 1650
-Text Notes 1800 2650 0    60   ~ 0
-Reset pin has a pull-up resistor.\nNo external one needed.
+	2300 1900 2050 1900
+NoConn ~ 2300 1800
 $EndSCHEMATC

Commit message: Added consistency between Schematic and Code
Parts:
- removed R12: 1k, projectLib:SMD-0805, symbol R
- added D2: LED GREEN, LEDs:LED_0603, symbol LED
- added R10: 220R, projectLib:SMD-0805, symbol R
- D3: footprint projectLib:LED_0603_PIPE -> LEDs:LED_0603
Connections:
- net UP is gone; now on net LEFT: P2.3, R4.2, R6.1
- net DGND: now also R8.2, D2.1 (K)
- net LEFT: no longer P2.6, R7.2, R8.1
- net G: now reaches IC1.5 (PB0(MOSI/DI/SDA/AIN0/OC0A/OC1A/AREF/PCINT0))
- net G: now also R10.1
- net CENTER: no longer names the net of P2.2
- net CENTER: no longer R8.2
- new net: D2.2 (A), R10.2
- new net RIGHT: P2.6, R7.2, R8.1
Other:
- note added: "Reset pin has a pull-up resistor.\nNo external one needed."
- note removed: "Reset pin has internal pull-up resistor.\nNo external one needed."
- moved on the sheet: D3, R11
Changed lines of the file:
@@
 Sheet 1 1
 Title "MemType PCB schematic"
-Date "2016-06-08"
-Rev "3"
+Date "2016-01-06"
+Rev "2"
 Comp "website: www.area0x33.com"
 Comment1 ""
@@
 $EndComp
 $Comp
-L DGND #PWR5
+L DGND #PWR01
 U 1 1 5432C0B8
 P 5100 2450
-F 0 "#PWR5" H 5100 2450 40  0001 C CNN
+F 0 "#PWR01" H 5100 2450 40  0001 C CNN
 F 1 "DGND" H 5100 2380 40  0000 C CNN
 F 2 "" H 5100 2450 60  0000 C CNN
@@
 $EndComp
 $Comp
-L +5V #PWR4
+L +5V #PWR02
 U 1 1 5432D97B
 P 5100 1650
-F 0 "#PWR4" H 5100 1740 20  0001 C CNN
+F 0 "#PWR02" H 5100 1740 20  0001 C CNN
 F 1 "+5V" H 5100 1740 30  0000 C CNN
 F 2 "" H 5100 1650 60  0000 C CNN
@@
 $EndComp
 $Comp
-L +5V #PWR1
+L +5V #PWR03
 U 1 1 5432D981
 P 1050 1350
-F 0 "#PWR1" H 1050 1440 20  0001 C CNN
+F 0 "#PWR03" H 1050 1440 20  0001 C CNN
 F 1 "+5V" H 1050 1440 30  0000 C CNN
 F 2 "" H 1050 1350 60  0000 C CNN
@@
 Connection ~ 1250 2100
 $Comp
-L DGND #PWR2
+L DGND #PWR04
 U 1 1 5432DBE1
 P 1150 2900
-F 0 "#PWR2" H 1150 2900 40  0001 C CNN
+F 0 "#PWR04" H 1150 2900 40  0001 C CNN
 F 1 "DGND" H 1150 2830 40  0000 C CNN
 F 2 "" H 1150 2900 60  0000 C CNN
@@
 	5800 1750 5800 1700
 $Comp
-L DGND #PWR7
+L DGND #PWR05
 U 1 1 5432DF65
 P 6000 1750
-F 0 "#PWR7" H 6000 1750 40  0001 C CNN
+F 0 "#PWR05" H 6000 1750 40  0001 C CNN
 F 1 "DGND" H 6000 1680 40  0000 C CNN
 F 2 "" H 6000 1750 60  0000 C CNN
@@
 $EndComp
 $Comp
-L +5V #PWR6
+L +5V #PWR06
 U 1 1 5432DF84
 P 5600 1750
-F 0 "#PWR6" H 5600 1840 20  0001 C CNN
+F 0 "#PWR06" H 5600 1840 20  0001 C CNN
 F 1 "+5V" H 5600 1840 30  0000 C CNN
 F 2 "" H 5600 1750 60  0000 C CNN
@@
 	8850 1250 8850 1200
 $Comp
-L +5V #PWR10
+L +5V #PWR07
 U 1 1 543DE636
 P 8850 1200
-F 0 "#PWR10" H 8850 1290 20  0001 C CNN
+F 0 "#PWR07" H 8850 1290 20  0001 C CNN
 F 1 "+5V" H 8850 1290 30  0000 C CNN
 F 2 "" H 8850 1200 60  0000 C CNN
@@
 	1    0    0    -1
 $EndComp
+Wire Wire Line
+	8850 3400 8850 3450
 Wire Wire Line
 	8850 2300 8650 2300
@@
 Microcontroller circuit and peripherals
 Wire Notes Line
-	6750 1050 6750 4100
-Wire Notes Line
-	9200 1050 9200 4100
+	6750 3700 9150 3700
+Wire Notes Line
+	6750 1050 6750 3700
+Wire Notes Line
+	9200 3700 9200 1050
 $Comp
 L ZENER_DUAL D1
@@
 	1050 2200 1050 2350
 $Comp
-L DGND #PWR9
+L DGND #PWR08
 U 1 1 546258D9
 P 8100 2600
-F 0 "#PWR9" H 8100 2600 40  0001 C CNN
+F 0 "#PWR08" H 8100 2600 40  0001 C CNN
 F 1 "DGND" H 8100 2530 40  0000 C CNN
 F 2 "" H 8100 2600 60  0000 C CNN
@@
 $EndComp
 $Comp
-L DGND #PWR11
+L DGND #PWR09
 U 1 1 5462598D
-P 8850 3900
-F 0 "#PWR11" H 8850 3900 40  0001 C CNN
-F 1 "DGND" H 8850 3830 40  0000 C CNN
-F 2 "" H 8850 3900 60  0000 C CNN
-F 3 "" H 8850 3900 60  0000 C CNN
-	1    8850 3900
+P 8850 3450
+F 0 "#PWR09" H 8850 3450 40  0001 C CNN
+F 1 "DGND" H 8850 3380 40  0000 C CNN
+F 2 "" H 8850 3450 60  0000 C CNN
+F 3 "" H 8850 3450 60  0000 C CNN
+	1    8850 3450
 	1    0    0    -1
 $EndComp
@@
 	8300 2850 8300 1450
 Text Label 7850 1950 0    60   ~ 0
-RIGHT
+UP
 Text Label 7850 1750 0    60   ~ 0
-UP
+LEFT
 Text Label 7850 1650 0    60   ~ 0
 DOWN
 Text Label 7850 1450 0    60   ~ 0
-LEFT
+RIGHT
 $Comp
 L R R9
@@
 	6450 2000 6250 2000
 $Comp
-L DGND #PWR8
+L DGND #PWR010
 U 1 1 568C63F8
 P 6250 2100
-F 0 "#PWR8" H 6250 2100 40  0001 C CNN
+F 0 "#PWR010" H 6250 2100 40  0001 C CNN
 F 1 "DGND" H 6250 2030 40  0000 C CNN
 F 2 "" H 6250 2100 60  0000 C CNN
@@
 Wire Wire Line
 	8400 1950 7850 1950
+NoConn ~ 7850 1850
 $Comp
 L USB_A P1
@@
 $EndComp
 $Comp
-L DGND #PWR3
+L LED D2
+U 1 1 56901E90
+P 3850 3350
+F 0 "D2" H 3850 3450 50  0000 C CNN
+F 1 "LED GREEN" H 3850 3250 50  0000 C CNN
+F 2 "LEDs:LED_0603" H 3850 3350 60  0001 C CNN
+F 3 "" H 3850 3350 60  0001 C CNN
+F 4 "L29K-F2J1-24-Z" H 3850 3350 60  0001 C CNN "mouser"
+	1    3850 3350
+	0    1    -1   0
+$EndComp
+$Comp
+L DGND #PWR011
 U 1 1 5690231F
-P 3750 3600
-F 0 "#PWR3" H 3750 3600 40  0001 C CNN
-F 1 "DGND" H 3750 3530 40  0000 C CNN
-F 2 "" H 3750 3600 60  0000 C CNN
-F 3 "" H 3750 3600 60  0000 C CNN
-	1    3750 3600
+P 3850 3700
+F 0 "#PWR011" H 3850 3700 40  0001 C CNN
+F 1 "DGND" H 3850 3630 40  0000 C CNN
+F 2 "" H 3850 3700 60  0000 C CNN
+F 3 "" H 3850 3700 60  0000 C CNN
+	1    3850 3700
 	1    0    0    -1
 $EndComp
@@
 L LED D3
 U 1 1 569024A8
-P 3750 3350
-F 0 "D3" H 3750 3450 50  0000 C CNN
-F 1 "LED RED" H 3750 3250 50  0000 C CNN
-F 2 "projectLib:LED_0603_PIPE" H 3750 3350 60  0001 C CNN
-F 3 "" H 3750 3350 60  0001 C CNN
-F 4 "Q976-NR-1" H 3750 3350 60  0001 C CNN "mouser"
-	1    3750 3350
+P 4150 3350
+F 0 "D3" H 4150 3450 50  0000 C CNN
+F 1 "LED RED" H 4150 3250 50  0000 C CNN
+F 2 "LEDs:LED_0603" H 4150 3350 60  0001 C CNN
+F 3 "" H 4150 3350 60  0001 C CNN
+F 4 "Q976-NR-1" H 4150 3350 60  0001 C CNN "mouser"
+	1    4150 3350
 	0    1    -1   0
 $EndComp
 Wire Wire Line
-	3750 3600 3750 3550
+	2300 1900 2050 1900
+Wire Wire Line
+	2300 1800 2050 1800
+Wire Wire Line
+	3850 3550 3850 3700
+Wire Wire Line
+	3850 3600 4150 3600
+Wire Wire Line
+	4150 3600 4150 3550
+Connection ~ 3850 3600
 $Comp
 L R R11
 U 1 1 569034B6
-P 3750 2850
-F 0 "R11" V 3750 2950 40  0000 C CNN
-F 1 "220R" V 3750 2800 40  0000 C CNN
-F 2 "projectLib:SMD-0805" V 3680 2850 30  0001 C CNN
-F 3 "~" H 3750 2850 30  0000 C CNN
-F 4 "1/8W" V 3750 2850 40  0001 C CNN "Power"
-F 5 "ERJ-6GEYJ221V" V 3750 2850 60  0001 C CNN "mouser"
-	1    3750 2850
-	1    0    0    -1
-$EndComp
-Wire Wire Line
-	3750 3100 3750 3150
-Text Label 3750 2600 0    60   ~ 0
+P 4150 2850
+F 0 "R11" V 4150 2950 40  0000 C CNN
+F 1 "220R" V 4150 2800 40  0000 C CNN
+F 2 "projectLib:SMD-0805" V 4080 2850 30  0001 C CNN
+F 3 "~" H 4150 2850 30  0000 C CNN
+F 4 "1/8W" V 4150 2850 40  0001 C CNN "Power"
+F 5 "ERJ-6GEYJ221V" V 4150 2850 60  0001 C CNN "mouser"
+	1    4150 2850
+	1    0    0    -1
+$EndComp
+$Comp
+L R R10
+U 1 1 5690360A
+P 3850 2850
+F 0 "R10" V 3850 2950 40  0000 C CNN
+F 1 "220R" V 3850 2800 40  0000 C CNN
+F 2 "projectLib:SMD-0805" V 3780 2850 30  0001 C CNN
+F 3 "~" H 3850 2850 30  0000 C CNN
+F 4 "1/8W" V 3850 2850 40  0001 C CNN "Power"
+F 5 "ERJ-6GEYJ221V" V 3850 2850 60  0001 C CNN "mouser"
+	1    3850 2850
+	1    0    0    -1
+$EndComp
+Wire Wire Line
+	4150 3100 4150 3150
+Wire Wire Line
+	3850 3100 3850 3150
+Text Label 4150 2600 0    60   ~ 0
+R
+Text Label 3850 2600 0    60   ~ 0
+G
+Text Label 2050 1800 0    60   ~ 0
+G
+Text Label 2050 1900 0    60   ~ 0
 R
 Wire Wire Line
 	5100 1800 5100 1650
 Text Notes 1800 2650 0    60   ~ 0
-Reset pin has internal pull-up resistor.\nNo external one needed.
-$Comp
-L R R12
-U 1 1 575737C3
-P 8850 3650
-F 0 "R12" V 8850 3750 40  0000 C CNN
-F 1 "1k" V 8850 3600 40  0000 C CNN
-F 2 "projectLib:SMD-0805" V 8780 3650 30  0001 C CNN
-F 3 "~" H 8850 3650 30  0000 C CNN
-F 4 "1/4W" V 8850 3650 40  0001 C CNN "Power"
-F 5 "ERJ-6GEYJ102V" V 8850 3650 60  0001 C CNN "mouser"
-	1    8850 3650
-	1    0    0    -1
-$EndComp
-Wire Notes Line
-	9200 4100 6750 4100
-Wire Wire Line
-	8850 3400 8500 3400
-Wire Wire Line
-	8500 3400 8500 1850
-Wire Wire Line
-	8500 1850 7850 1850
-Text Label 7850 1850 0    60   ~ 0
-CENTER
-Text Label 2050 1900 0    60   ~ 0
-R
-Wire Wire Line
-	2300 1900 2050 1900
-NoConn ~ 2300 1800
+Reset pin has a pull-up resistor.\nNo external one needed.
 $EndSCHEMATC

Commit message: memtype hardware revision 2.1
Parts:
- D2, D3: footprint LEDs:LED_0603 -> projectLib:LED_0603_PIPE
Changed lines of the file:
@@
 F 0 "D2" H 3850 3450 50  0000 C CNN
 F 1 "LED GREEN" H 3850 3250 50  0000 C CNN
-F 2 "LEDs:LED_0603" H 3850 3350 60  0001 C CNN
+F 2 "projectLib:LED_0603_PIPE" H 3850 3350 60  0001 C CNN
 F 3 "" H 3850 3350 60  0001 C CNN
 F 4 "L29K-F2J1-24-Z" H 3850 3350 60  0001 C CNN "mouser"
@@
 F 0 "D3" H 4150 3450 50  0000 C CNN
 F 1 "LED RED" H 4150 3250 50  0000 C CNN
-F 2 "LEDs:LED_0603" H 4150 3350 60  0001 C CNN
+F 2 "projectLib:LED_0603_PIPE" H 4150 3350 60  0001 C CNN
 F 3 "" H 4150 3350 60  0001 C CNN
 F 4 "Q976-NR-1" H 4150 3350 60  0001 C CNN "mouser"
